Commit message: not woek

File: src/iris_robot_description/urdf/iris_robot.xacro (robot description, xacro)
@@ -6,5 +6,5 @@
 <link name="base_link">
   <inertial>
-    <origin xyz="0.1997829135981424 0.07174507294677275 -0.03318689491945889" rpy="0 0 0"/>
+    <origin xyz="0.1831445962056383 0.07239617157428578 0.027463824756232526" rpy="0 0 0"/>
     <mass value="3.7613399363810003"/>
     <inertia ixx="0.074761" iyy="0.07222" izz="0.145535" ixy="0.006375" iyz="0.003562" ixz="3.1e-05"/>
@@ -15,5 +15,5 @@
       <mesh filename="package://iris_robot_description/meshes/base_link.stl" scale="0.001 0.001 0.001"/>
     </geometry>
-    <material name="silver"/>
+    <material name="black"/>
   </visual>
   <collision>
@@ -26,10 +26,10 @@
 <link name="left_motor_bracket_1">
   <inertial>
-    <origin xyz="-0.051697526696497936 -0.0009996854268710664 0.049488279937635715" rpy="0 0 0"/>
+    <origin xyz="-0.05169784408900585 -0.0009995867993597696 0.04948899961332788" rpy="0 0 0"/>
     <mass value="0.47321750244262606"/>
     <inertia ixx="0.000634" iyy="0.000857" izz="0.000382" ixy="-9e-05" iyz="0.0" ixz="-4e-06"/>
   </inertial>
   <visual>
-    <origin xyz="-0.298167 0.092634 0.02819" rpy="0 0 0"/>
+    <origin xyz="-0.281529 0.091983 -0.03246" rpy="0 0 0"/>
     <geometry>
       <mesh filename="package://iris_robot_description/meshes/left_motor_bracket_1.stl" scale="0.001 0.001 0.001"/>
@@ -38,5 +38,5 @@
   </visual>
   <collision>
-    <origin xyz="-0.298167 0.092634 0.02819" rpy="0 0 0"/>
+    <origin xyz="-0.281529 0.091983 -0.03246" rpy="0 0 0"/>
     <geometry>
       <mesh filename="package://iris_robot_description/meshes/left_motor_bracket_1.stl" scale="0.001 0.001 0.001"/>
@@ -46,10 +46,10 @@
 <link name="left_motor_1">
   <inertial>
-    <origin xyz="-0.0208545067980154 0.05897406854688668 -0.0028576079823523295" rpy="0 0 0"/>
+    <origin xyz="-0.020854824190523702 0.05897416717439771 -0.0028578883066602556" rpy="0 0 0"/>
     <mass value="0.3401593265595349"/>
     <inertia ixx="0.000387" iyy="0.000201" izz="0.000434" ixy="7.5e-05" iyz="1.1e-05" ixz="-4e-06"/>
   </inertial>
   <visual>
-    <origin xyz="-0.242374 0.080585 -0.046939" rpy="0 0 0"/>
+    <origin xyz="-0.225736 0.079934 -0.10759" rpy="0 0 0"/>
     <geometry>
       <mesh filename="package://iris_robot_description/meshes/left_motor_1.stl" scale="0.001 0.001 0.001"/>
@@ -58,5 +58,5 @@
   </visual>
   <collision>
-    <origin xyz="-0.242374 0.080585 -0.046939" rpy="0 0 0"/>
+    <origin xyz="-0.225736 0.079934 -0.10759" rpy="0 0 0"/>
     <geometry>
       <mesh filename="package://iris_robot_description/meshes/left_motor_1.stl" scale="0.001 0.001 0.001"/>
@@ -66,10 +66,10 @@
 <link name="left_motor_ash_1">
   <inertial>
-    <origin xyz="0.016048832983915545 -0.04538293390535532 0.0021989546019030755" rpy="0 0 0"/>
+    <origin xyz="0.01604851559157805 -0.04538283527782078 0.002199674276821953" rpy="0 0 0"/>
     <mass value="0.08025811044162247"/>
     <inertia ixx="5.8e-05" iyy="9e-06" izz="6.4e-05" ixy="2e-05" iyz="3e-06" ixz="-1e-06"/>
   </inertial>
   <visual>
-    <origin xyz="-0.241279 0.079754 -0.006352" rpy="0 0 0"/>
+    <origin xyz="-0.224641 0.079103 -0.067002" rpy="0 0 0"/>
     <geometry>
       <mesh filename="package://iris_robot_description/meshes/left_motor_ash_1.stl" scale="0.001 0.001 0.001"/>
@@ -78,5 +78,5 @@
   </visual>
   <collision>
-    <origin xyz="-0.241279 0.079754 -0.006352" rpy="0 0 0"/>
+    <origin xyz="-0.224641 0.079103 -0.067002" rpy="0 0 0"/>
     <geometry>
       <mesh filename="package://iris_robot_description/meshes/left_motor_ash_1.stl" scale="0.001 0.001 0.001"/>
@@ -86,10 +86,10 @@
 <link name="left_motor_bracket_cover_1">
   <inertial>
-    <origin xyz="-0.02438125526712065 -0.013054566739830922 -0.024735734973780357" rpy="0 0 0"/>
+    <origin xyz="-0.024381572659628287 -0.013054468112319514 -0.02473601529808811" rpy="0 0 0"/>
     <mass value="0.0769306560962844"/>
     <inertia ixx="3.3e-05" iyy="5.6e-05" izz="3.1e-05" ixy="-9e-06" iyz="-1e-06" ixz="0.0"/>
   </inertial>
   <visual>
-    <origin xyz="-0.278335 0.102459 -0.034286" rpy="0 0 0"/>
+    <origin xyz="-0.261697 0.101808 -0.094937" rpy="0 0 0"/>
     <geometry>
       <mesh filename="package://iris_robot_description/meshes/left_motor_bracket_cover_1.stl" scale="0.001 0.001 0.001"/>
@@ -98,5 +98,5 @@
   </visual>
   <collision>
-    <origin xyz="-0.278335 0.102459 -0.034286" rpy="0 0 0"/>
+    <origin xyz="-0.261697 0.101808 -0.094937" rpy="0 0 0"/>
     <geometry>
       <mesh filename="package://iris_robot_description/meshes/left_motor_bracket_cover_1.stl" scale="0.001 0.001 0.001"/>
@@ -106,10 +106,10 @@
 <link name="left_ash_to_omni_connector_front_1">
   <inertial>
-    <origin xyz="-0.006616919145590983 0.018712163153787126 -0.0009071806635806701" rpy="0 0 0"/>
+    <origin xyz="-0.006617236538144222 0.01871226178128013 -0.0009064609879057689" rpy="0 0 0"/>
     <mass value="0.1791480879958417"/>
     <inertia ixx="5.8e-05" iyy="6.4e-05" izz="5.8e-05" ixy="-2e-06" iyz="-0.0" ixz="0.0"/>
   </inertial>
   <visual>
-    <origin xyz="-0.273751 0.17158 -0.010802" rpy="0 0 0"/>
+    <origin xyz="-0.257113 0.170929 -0.071452" rpy="0 0 0"/>
     <geometry>
       <mesh filename="package://iris_robot_description/meshes/left_ash_to_omni_connector_front_1.stl" scale="0.001 0.001 0.001"/>
@@ -118,5 +118,5 @@
   </visual>
   <collision>
-    <origin xyz="-0.273751 0.17158 -0.010802" rpy="0 0 0"/>
+    <origin xyz="-0.257113 0.170929 -0.071452" rpy="0 0 0"/>
     <geometry>
       <mesh filename="package://iris_robot_description/meshes/left_ash_to_omni_connector_front_1.stl" scale="0.001 0.001 0.001"/>
@@ -126,10 +126,10 @@
 <link name="front_right_omni_1">
   <inertial>
-    <origin xyz="-0.0025565844279144545 -0.00362987882889354 -0.023379755452968526" rpy="0 0 0"/>
+    <origin xyz="-0.01942590182350401 -0.008966780202215252 -0.010418035771954784" rpy="0 0 0"/>
     <mass value="0.23500963441195055"/>
     <inertia ixx="0.000307" iyy="0.000518" izz="0.000278" ixy="-8.5e-05" iyz="-1.2e-05" ixz="4e-06"/>
   </inertial>
   <visual>
-    <origin xyz="-0.274809 0.163712 -0.033976" rpy="0 0 0"/>
+    <origin xyz="-0.27504 0.157724 -0.081665" rpy="0 0 0"/>
     <geometry>
       <mesh filename="package://iris_robot_description/meshes/front_right_omni_1.stl" scale="0.001 0.001 0.001"/>
@@ -138,5 +138,5 @@
   </visual>
   <collision>
-    <origin xyz="-0.274809 0.163712 -0.033976" rpy="0 0 0"/>
+    <origin xyz="-0.27504 0.157724 -0.081665" rpy="0 0 0"/>
     <geometry>
       <mesh filename="package://iris_robot_description/meshes/front_right_omni_1.stl" scale="0.001 0.001 0.001"/>
@@ -146,10 +146,10 @@
 <link name="mid_right_omni_1">
   <inertial>
-    <origin xyz="-0.02150992431476545 -0.006449952818261606 -0.009005428134492715" rpy="0 0 0"/>
+    <origin xyz="-0.01973886434902064 -0.0047501977858498134 0.013159920747479098" rpy="0 0 0"/>
     <mass value="0.2348808094813233"/>
     <inertia ixx="0.000307" iyy="0.000518" izz="0.000278" ixy="-8.5e-05" iyz="-1.2e-05" ixz="4e-06"/>
   </inertial>
   <visual>
-    <origin xyz="-0.286499 0.141226 -0.018298" rpy="0 0 0"/>
+    <origin xyz="-0.267934 0.142311 -0.057169" rpy="0 0 0"/>
     <geometry>
       <mesh filename="package://iris_robot_description/meshes/mid_right_omni_1.stl" scale="0.001 0.001 0.001"/>
@@ -158,5 +158,5 @@
   </visual>
   <collision>
-    <origin xyz="-0.286499 0.141226 -0.018298" rpy="0 0 0"/>
+    <origin xyz="-0.267934 0.142311 -0.057169" rpy="0 0 0"/>
     <geometry>
       <mesh filename="package://iris_robot_description/meshes/mid_right_omni_1.stl" scale="0.001 0.001 0.001"/>
@@ -166,10 +166,10 @@
 <link name="left_ash_to_omni_connector_rear_1">
   <inertial>
-    <origin xyz="-0.02648735023287563 -3.924698516621916e-05 -0.004728931951233606" rpy="0 0 0"/>
+    <origin xyz="-0.020120484439436953 0.0032920238285845393 0.017557937881550634" rpy="0 0 0"/>
     <mass value="0.09595762654106495"/>
     <inertia ixx="3.2e-05" iyy="5.1e-05" izz="2.9e-05" ixy="-8e-06" iyz="-1e-06" ixz="0.0"/>
   </inertial>
   <visual>
-    <origin xyz="-0.286721 0.138277 -0.011804" rpy="0 0 0"/>
+    <origin xyz="-0.262736 0.141195 -0.05241" rpy="0 0 0"/>
     <geometry>
       <mesh filename="package://iris_robot_description/meshes/left_ash_to_omni_connector_rear_1.stl" scale="0.001 0.001 0.001"/>
@@ -178,5 +178,5 @@
   </visual>
   <collision>
-    <origin xyz="-0.286721 0.138277 -0.011804" rpy="0 0 0"/>
+    <origin xyz="-0.262736 0.141195 -0.05241" rpy="0 0 0"/>
     <geometry>
       <mesh filename="package://iris_robot_description/meshes/left_ash_to_omni_connector_rear_1.stl" scale="0.001 0.001 0.001"/>
@@ -186,10 +186,10 @@
 <link name="rear_right_omni_1">
   <inertial>
-    <origin xyz="-0.02221384333561427 -0.00652934620012538 -0.005498715058939618" rpy="0 0 0"/>
+    <origin xyz="-0.017440703587482093 -0.0038125251946335426 0.015735515057858036" rpy="0 0 0"/>
     <mass value="0.23500963441194936"/>
     <inertia ixx="0.000307" iyy="0.000518" izz="0.000278" ixy="-8.5e-05" iyz="-1.2e-05" ixz="4e-06"/>
   </inertial>
   <visual>
-    <origin xyz="-0.277582 0.122305 -0.013681" rpy="0 0 0"/>
+    <origin xyz="-0.256983 0.123951 -0.05583" rpy="0 0 0"/>
     <geometry>
       <mesh filename="package://iris_robot_description/meshes/rear_right_omni_1.stl" scale="0.001 0.001 0.001"/>
@@ -198,5 +198,5 @@
   </visual>
   <collision>
-    <origin xyz="-0.277582 0.122305 -0.013681" rpy="0 0 0"/>
+    <origin xyz="-0.256983 0.123951 -0.05583" rpy="0 0 0"/>
     <geometry>
       <mesh filename="package://iris_robot_description/meshes/rear_right_omni_1.stl" scale="0.001 0.001 0.001"/>
@@ -206,10 +206,10 @@
 <link name="rear_motor_bracket_1">
   <inertial>
-    <origin xyz="-0.031387654658413866 0.04246961585948514 0.04729811610200291" rpy="0 0 0"/>
+    <origin xyz="-0.0313879720509227 0.04246971448699596 0.04729783577769485" rpy="0 0 0"/>
     <mass value="0.47321750244279526"/>
     <inertia ixx="0.000723" iyy="0.000764" izz="0.000386" ixy="0.00014" iyz="-3.8e-05" ixz="-2.4e-05"/>
   </inertial>
   <visual>
-    <origin xyz="-0.329052 -0.138527 0.039659" rpy="0 0 0"/>
+    <origin xyz="-0.312414 -0.139178 -0.020992" rpy="0 0 0"/>
     <geometry>
       <mesh filename="package://iris_robot_description/meshes/rear_motor_bracket_1.stl" scale="0.001 0.001 0.001"/>
@@ -218,5 +218,5 @@
   </visual>
   <collision>
-    <origin xyz="-0.329052 -0.138527 0.039659" rpy="0 0 0"/>
+    <origin xyz="-0.312414 -0.139178 -0.020992" rpy="0 0 0"/>
     <geometry>
       <mesh filename="package://iris_robot_description/meshes/rear_motor_bracket_1.stl" scale="0.001 0.001 0.001"/>
@@ -226,10 +226,10 @@
 <link name="rear_motor_bracket_cover_1">
   <inertial>
-    <origin xyz="-0.01849719969034308 0.018509146826390682 -0.026305410316676468" rpy="0 0 0"/>
+    <origin xyz="-0.01849751708285191 0.018509245453901563 -0.026305690640984522" rpy="0 0 0"/>
     <mass value="0.07693065609628418"/>
     <inertia ixx="4.2e-05" iyy="4.7e-05" izz="3.1e-05" ixy="1.5e-05" iyz="-1e-06" ixz="-1e-06"/>
   </inertial>
   <visual>
-    <origin xyz="-0.330799 -0.17898 -0.020288" rpy="0 0 0"/>
+    <origin xyz="-0.314161 -0.179631 -0.080939" rpy="0 0 0"/>
     <geometry>
       <mesh filename="package://iris_robot_description/meshes/rear_motor_bracket_cover_1.stl" scale="0.001 0.001 0.001"/>
@@ -238,5 +238,5 @@
   </visual>
   <collision>
-    <origin xyz="-0.330799 -0.17898 -0.020288" rpy="0 0 0"/>
+    <origin xyz="-0.314161 -0.179631 -0.080939" rpy="0 0 0"/>
     <geometry>
       <mesh filename="package://iris_robot_description/meshes/rear_motor_bracket_cover_1.stl" scale="0.001 0.001 0.001"/>
@@ -246,10 +246,10 @@
 <link name="rear_motor_1">
   <inertial>
-    <origin xyz="-0.03420629073321296 -0.039930650909949156 0.0020492661372191606" rpy="0 0 0"/>
+    <origin xyz="-0.034205608125721654 -0.03993055228243836 0.002048985812911089" rpy="0 0 0"/>
     <mass value="0.3401593265595337"/>
     <inertia ixx="0.000312" iyy="0.000276" izz="0.000435" ixy="-0.000118" iyz="8e-06" ixz="6e-06"/>
   </inertial>
   <visual>
-    <origin xyz="-0.289612 -0.172816 -0.034336" rpy="0 0 0"/>
+    <origin xyz="-0.272973 -0.173467 -0.094987" rpy="0 0 0"/>
     <geometry>
       <mesh filename="package://iris_robot_description/meshes/rear_motor_1.stl" scale="0.001 0.001 0.001"/>
@@ -258,5 +258,5 @@
   </visual>
   <collision>
-    <origin xyz="-0.289612 -0.172816 -0.034336" rpy="0 0 0"/>
+    <origin xyz="-0.272973 -0.173467 -0.094987" rpy="0 0 0"/>
     <geometry>
       <mesh filename="package://iris_robot_description/meshes/rear_motor_1.stl" scale="0.001 0.001 0.001"/>
@@ -266,10 +266,10 @@
 <link name="rear_motor_ash_1">
   <inertial>
-    <origin xyz="0.03132504925632934 0.03656813129600975 -0.0018765445552491305" rpy="0 0 0"/>
+    <origin xyz="0.03132573186382048 0.03656822992352057 -0.001876824879557197" rpy="0 0 0"/>
     <mass value="0.0802581104416225"/>
     <inertia ixx="3.8e-05" iyy="2.8e-05" izz="6.4e-05" ixy="-3.1e-05" iyz="2e-06" ixz="2e-06"/>
   </inertial>
   <visual>
-    <origin xyz="-0.287566 -0.168545 0.005998" rpy="0 0 0"/>
+    <origin xyz="-0.270927 -0.169196 -0.054653" rpy="0 0 0"/>
     <geometry>
       <mesh filename="package://iris_robot_description/meshes/rear_motor_ash_1.stl" scale="0.001 0.001 0.001"/>
@@ -278,5 +278,5 @@
   </visual>
   <collision>
-    <origin xyz="-0.287566 -0.168545 0.005998" rpy="0 0 0"/>
+    <origin xyz="-0.270927 -0.169196 -0.054653" rpy="0 0 0"/>
     <geometry>
       <mesh filename="package://iris_robot_description/meshes/rear_motor_ash_1.stl" scale="0.001 0.001 0.001"/>
@@ -286,10 +286,10 @@
 <link name="rear_ash_to_omni_connector_rear_1">
   <inertial>
-    <origin xyz="-0.012915908038877266 -0.015077361998288241 0.0007737419278990767" rpy="0 0 0"/>
+    <origin xyz="-0.012916225431386319 -0.015077263370777416 0.0007734616035909858" rpy="0 0 0"/>
     <mass value="0.17914808799583984"/>
     <inertia ixx="6.1e-05" iyy="6.2e-05" izz="5.8e-05" ixy="3e-06" iyz="-0.0" ixz="-0.0"/>
   </inertial>
   <visual>
-    <origin xyz="-0.350948 -0.242535 0.009795" rpy="0 0 0"/>
+    <origin xyz="-0.33431 -0.243186 -0.050856" rpy="0 0 0"/>
     <geometry>
       <mesh filename="package://iris_robot_description/meshes/rear_ash_to_omni_connector_rear_1.stl" scale="0.001 0.001 0.001"/>
@@ -298,5 +298,5 @@
   </visual>
   <collision>
-    <origin xyz="-0.350948 -0.242535 0.009795" rpy="0 0 0"/>
+    <origin xyz="-0.33431 -0.243186 -0.050856" rpy="0 0 0"/>
     <geometry>
       <mesh filename="package://iris_robot_description/meshes/rear_ash_to_omni_connector_rear_1.stl" scale="0.001 0.001 0.001"/>
@@ -306,10 +306,10 @@
 <link name="front_rear_omni_1">
   <inertial>
-    <origin xyz="-0.005150311755604486 0.005227270431975128 -0.02263778094796189" rpy="0 0 0"/>
+    <origin xyz="-0.005150629148113484 0.005227369059485898 -0.022637061272269964" rpy="0 0 0"/>
     <mass value="0.23500963441722925"/>
     <inertia ixx="0.000392" iyy="0.000433" izz="0.000277" ixy="0.000134" iyz="-8e-06" ixz="-7e-06"/>
   </inertial>
   <visual>
-    <origin xyz="-0.353173 -0.233893 -0.013018" rpy="0 0 0"/>
+    <origin xyz="-0.336535 -0.234544 -0.073668" rpy="0 0 0"/>
     <geometry>
       <mesh filename="package://iris_robot_description/meshes/front_rear_omni_1.stl" scale="0.001 0.001 0.001"/>
@@ -318,5 +318,5 @@
   </visual>
   <collision>
-    <origin xyz="-0.353173 -0.233893 -0.013018" rpy="0 0 0"/>
+    <origin xyz="-0.336535 -0.234544 -0.073668" rpy="0 0 0"/>
     <geometry>
       <mesh filename="package://iris_robot_description/meshes/front_rear_omni_1.stl" scale="0.001 0.001 0.001"/>
@@ -326,10 +326,10 @@
 <link name="mid_rear_omni_1">
   <inertial>
-    <origin xyz="-0.0009649619788453245 -0.0011463945353487603 6.0714852895216165e-05" rpy="0 0 0"/>
+    <origin xyz="-0.0009652793713543217 -0.0011462959078379353 6.143452858713844e-05" rpy="0 0 0"/>
     <mass value="0.23488080945950318"/>
     <inertia ixx="0.000392" iyy="0.000433" izz="0.000277" ixy="0.000134" iyz="-8e-06" ixz="-7e-06"/>
   </inertial>
   <visual>
-    <origin xyz="-0.335346 -0.224322 0.00886" rpy="0 0 0"/>
+    <origin xyz="-0.318708 -0.224973 -0.05179" rpy="0 0 0"/>
     <geometry>
       <mesh filename="package://iris_robot_description/meshes/mid_rear_omni_1.stl" scale="0.001 0.001 0.001"/>
@@ -338,5 +338,5 @@
   </visual>
   <collision>
-    <origin xyz="-0.335346 -0.224322 0.00886" rpy="0 0 0"/>
+    <origin xyz="-0.318708 -0.224973 -0.05179" rpy="0 0 0"/>
     <geometry>
       <mesh filename="package://iris_robot_description/meshes/mid_rear_omni_1.stl" scale="0.001 0.001 0.001"/>
@@ -346,10 +346,10 @@
 <link name="rear_ash_to_omni_connector_2_rear_1">
   <inertial>
-    <origin xyz="-0.00582885210636136 -0.006848352832746291 0.00035850381916479636" rpy="0 0 0"/>
+    <origin xyz="-0.005829169498870246 -0.006848254205235438 0.0003582234948567159" rpy="0 0 0"/>
     <mass value="0.09595762654117547"/>
     <inertia ixx="3.9e-05" iyy="4.3e-05" izz="2.9e-05" ixy="1.2e-05" iyz="-1e-06" ixz="-1e-06"/>
   </inertial>
   <visual>
-    <origin xyz="-0.332096 -0.220528 0.008666" rpy="0 0 0"/>
+    <origin xyz="-0.315458 -0.221179 -0.051985" rpy="0 0 0"/>
     <geometry>
       <mesh filename="package://iris_robot_description/meshes/rear_ash_to_omni_connector_2_rear_1.stl" scale="0.001 0.001 0.001"/>
@@ -358,5 +358,5 @@
   </visual>
   <collision>
-    <origin xyz="-0.332096 -0.220528 0.008666" rpy="0 0 0"/>
+    <origin xyz="-0.315458 -0.221179 -0.051985" rpy="0 0 0"/>
     <geometry>
       <mesh filename="package://iris_robot_description/meshes/rear_ash_to_omni_connector_2_rear_1.stl" scale="0.001 0.001 0.001"/>
@@ -366,10 +366,10 @@
 <link name="rear_rear_omni_1">
   <inertial>
-    <origin xyz="-0.0009755939810011105 -0.0011380856359286262 5.8802313065485154e-05" rpy="0 0 0"/>
+    <origin xyz="-0.0009749113735100234 -0.001137987008417829 5.8521988757449794e-05" rpy="0 0 0"/>
     <mass value="0.23500963441722744"/>
     <inertia ixx="0.000392" iyy="0.000433" izz="0.000277" ixy="0.000134" iyz="-8e-06" ixz="-7e-06"/>
   </inertial>
   <visual>
-    <origin xyz="-0.320395 -0.206868 0.007965" rpy="0 0 0"/>
+    <origin xyz="-0.303756 -0.207519 -0.052686" rpy="0 0 0"/>
     <geometry>
       <mesh filename="package://iris_robot_description/meshes/rear_rear_omni_1.stl" scale="0.001 0.001 0.001"/>
@@ -378,5 +378,5 @@
   </visual>
   <collision>
-    <origin xyz="-0.320395 -0.206868 0.007965" rpy="0 0 0"/>
+    <origin xyz="-0.303756 -0.207519 -0.052686" rpy="0 0 0"/>
     <geometry>
       <mesh filename="package://iris_robot_description/meshes/rear_rear_omni_1.stl" scale="0.001 0.001 0.001"/>
@@ -386,10 +386,10 @@
 <link name="right_motor_bracket_1">
   <inertial>
-    <origin xyz="-0.0005450198967092146 0.05334564740454088 0.04668862967935976" rpy="0 0 0"/>
+    <origin xyz="-0.0005443372892179228 0.05334574603205128 0.046688349355051714" rpy="0 0 0"/>
     <mass value="0.4732175024428434"/>
     <inertia ixx="0.000878" iyy="0.000611" izz="0.000384" ixy="-5e-05" iyz="-1.6e-05" ixz="2.5e-05"/>
   </inertial>
   <visual>
-    <origin xyz="-0.03448 -0.034651 0.033842" rpy="0 0 0"/>
+    <origin xyz="-0.017841 -0.035302 -0.026809" rpy="0 0 0"/>
     <geometry>
       <mesh filename="package://iris_robot_description/meshes/right_motor_bracket_1.stl" scale="0.001 0.001 0.001"/>
@@ -398,5 +398,5 @@
   </visual>
   <collision>
-    <origin xyz="-0.03448 -0.034651 0.033842" rpy="0 0 0"/>
+    <origin xyz="-0.017841 -0.035302 -0.026809" rpy="0 0 0"/>
     <geometry>
       <mesh filename="package://iris_robot_description/meshes/right_motor_bracket_1.stl" scale="0.001 0.001 0.001"/>
@@ -406,10 +406,10 @@
 <link name="right_motor_1">
   <inertial>
-    <origin xyz="0.05175533655903638 -0.00965162070469977 0.000337872160931979" rpy="0 0 0"/>
+    <origin xyz="0.051756019166527736 -0.009651522077189181 0.000337591836623935" rpy="0 0 0"/>
     <mass value="0.33990296538909626"/>
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